File: voltage_regulator.sch (EAGLE design)
At the start: 5 parts

Commit message: Add files via upload
Parts:
- removed LED1: Power_Status, led:NFSG036BT
- removed LM1117-3.3: 3.3V Regulator, linear:317EMP
- removed R1: 100, rcl:R-US_R0805
- added IC1: L4931D, v-reg-3:L4931D
- added LED2: Power_Status, led:NFSG036BT
- added R2: 330, rcl:R-US_R0805
- C1: value 10uF -> .1uF
- C2: value 100uF -> 2.2uF
Connections:
- removed net N$2: C2.1, LM1117-3.3.VO, R1.1
- removed net N$4: LED1.A, R1.2
- removed net N$8: C1.1, LM1117-3.3.VI
- new net 3.3V: C2.1, IC1.VOUT, R2.2
- new net N$1: LED2.A, R2.1
- new net N$5: C1.1, IC1.VIN
- net GND: now also IC1.GND, LED2.C; no longer LED1.C, LM1117-3.3.ADJ
Other:
- moved on the sheet: C1, C2
